File: Hardware/High Side VIN/SparkFun_XBee_Arduino_Shield_Qwiic.brd (EAGLE design)
At the start: 53.3 x 59.7 mm, 176 parts, among them J4 QWIIC_RIGHT_ANGLE, Q1 20V/4.2A/52mΩ/1.4W, Q2 20V/4.2A/52mΩ/1.4W, Q3 3.1A/30V/105mΩ, Q4 5.8A/30V/35mΩ, Q5 20V/4.2A/52mΩ/1.4W, U1 FSUSB30MUX_MSOP10, U2 AP63203, U3 ESD Diode, U4 FT231XS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

Commit message: Adds some rough drafts
Parts:
- removed C17, C18: 0.1uF, SparkFun-Capacitors:0603
- removed JP3: JUMPER-SMT_3_NO_SILK, SparkFun-Jumpers:SMT-JUMPER_3_NO_SILK
- removed Q1: 20V/4.2A/52mΩ/1.4W, SparkFun-DiscreteSemi:SOT23-3
- removed Q4: 5.8A/30V/35mΩ, SparkFun-DiscreteSemi:SOT23-3
- removed R23, R5: 10k, SparkFun-Resistors:0603
- removed U6: TXS0108, SparkFun-IC-Comms:VFQFN-20
- added D8: 3A/40V/500mV, SparkFun-DiscreteSemi:SMA-DIODE
- D7: value 3A/10V/280mV -> 3A/40V/500mV; device SparkFun-DiscreteSemi:SOD-323 -> SparkFun-DiscreteSemi:SMA-DIODE
- S4: value SWITCH_DP3T -> (none); device DP3T:SWITCH_DP3T_SMD_JWING -> SparkFun-Switches:SWITCH_DPDT_SMD_AYZ0202
- moved S4 104.0 mm to (-26.7, -43.2), turned to 0 degrees
- moved D7 97.7 mm to (-27.9, -54.6), turned to 0 degrees
Connections:
- removed net GATE: Q1.1, Q2.1, Q4.3, R23.2
- removed net IOREF: B1.IOREF, C18.1, JP3.2, U6.19
- removed net N$22: Q4.1, S4.P3, S4.P7
- removed net OE_BUS: B1.D3, R5.2, U6.10
- removed net SOURCE: Q1.2, Q2.2, R23.1
- new net N$18: D8.A, Q2.3
- new net N$9: Q2.1, S4.2, S4.5
- net 3.3V: no longer C17.1, JP3.1, U6.2
- net 5V: no longer JP3.3
- net D0: no longer U6.5
- net D0-TRANS: no longer U6.16
- net D1/SCL: no longer U6.1
- net D1/SCL-TRANS: no longer U6.20
- net D11/SDA: no longer U6.3
- net D11/SDA-TRANS: no longer U6.18
- net D13/TXO: no longer U6.9
- net D13/TXO-TRANS: no longer U6.12
- net D14/RXI: no longer U6.8
- net D14/RXI-TRANS: no longer U6.13
- net D9/!SLEEP!: no longer U6.4
- net D9/!SLEEP!-TRANS: no longer U6.17
- net GND: now also S4.1, S4.4; no longer C17.2, C18.2, Q4.2, R5.1, S4.P2, S4.P6, U6.11, U6.EPAD
- net VIN: now also Q2.2, S4.3, S4.6; no longer Q1.3, S4.P4, S4.P8
- net VIN_R3: now also D8.C; no longer Q2.3, S4.P1, S4.P5
Routing:
- net IOREF: track 53.1 -> 0.00 mm, vias 1 -> 0
- net VIN: track 41.2 -> 0.00 mm, vias 4 -> 0
- net GATE: track 18.0 -> 0.00 mm, vias 2 -> 0
- net OE_BUS: track 15.8 -> 0.00 mm, vias 1 -> 0
- net N$22: track 10.1 -> 0.00 mm
- net D1/SCL-TRANS: track 24.1 -> 16.0 mm
- net VIN_R3: track 10.9 -> 3.86 mm
- net 3.3V: track 22.2 -> 17.0 mm, vias 15 -> 12
- net 5V: track 6.83 -> 4.24 mm
- net D11/SDA: track 54.2 -> 51.8 mm
- net D9/!SLEEP!: track 34.5 -> 32.4 mm
- net D14/RXI-TRANS: track 20.0 -> 18.3 mm
- net D0-TRANS: track 14.6 -> 13.1 mm
- net GND: track 10.2 -> 8.75 mm, vias 106 -> 105
- net D0: track 93.7 -> 92.2 mm
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