File: Hardware/High Side VIN/SparkFun_XBee_Arduino_Shield_Qwiic.sch (EAGLE design)
At the start: 82 parts, among them J4 QWIIC_RIGHT_ANGLE, Q1 20V/4.2A/52mΩ/1.4W, Q2 20V/4.2A/52mΩ/1.4W, Q3 3.1A/30V/105mΩ, Q4 5.8A/30V/35mΩ, Q5 20V/4.2A/52mΩ/1.4W, U1 FSUSB30MUX_MSOP10, U2 AP63203, U3 ESD Diode, U4 FT231XS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

Commit message: Adds some rough drafts
Parts:
- removed C17, C18: 0.1uF, SparkFun-Capacitors:0.1UF-0603-25V-(+80/-20%)
- removed JP3: JUMPER-SMT_3_NO_SILK, SparkFun-Jumpers:JUMPER-SMT_3_NO_SILK
- removed Q1: 20V/4.2A/52mΩ/1.4W, SparkFun-DiscreteSemi:MOSFET_PCH-DMG2305UX-7
- removed Q4: 5.8A/30V/35mΩ, SparkFun-DiscreteSemi:MOSFET-NCH-AO3404A
- removed R23, R5: 10k, SparkFun-Resistors:10KOHM-0603-1/10W-1%
- removed U6: TXS0108, SparkFun-IC-Comms:TXS0108-VFQFN_20
- added D8: 3A/40V/500mV, SparkFun-DiscreteSemi:DIODE-SCHOTTKY-B340A
- D7: value 3A/10V/280mV -> 3A/40V/500mV; device SparkFun-DiscreteSemi:DIODE-SCHOTTKY-BAT60A -> SparkFun-DiscreteSemi:DIODE-SCHOTTKY-B340A
- S4: value SWITCH_DP3T -> (none); device DP3T:SWITCH_DP3T -> SparkFun-Switches:SWITCH-DPDT-SMD-AYZ0202
Connections:
- removed net GATE: Q1.G, Q2.G, Q4.D, R23.2
- removed net IOREF: B1.IOREF, C18.1, JP3.2, U6.VCCB
- removed net N$22: Q4.G, S4.3, S4.7
- removed net OE_BUS: B1.*D3, R5.2, U6.OE
- removed net SOURCE: Q1.S, Q2.S, R23.1
- new net N$18: D8.A, Q2.D
- new net N$9: Q2.G, S4.2, S4.5
- net 3.3V: no longer C17.1, JP3.1, U6.VCCA
- net 5V: no longer JP3.3
- net D0: no longer U6.A4
- net D0-TRANS: no longer U6.B4
- net D1/SCL: no longer U6.A1
- net D1/SCL-TRANS: no longer U6.B1
- net D11/SDA: no longer U6.A2
- net D11/SDA-TRANS: no longer U6.B2
- net D13/TXO: no longer U6.A8
- net D13/TXO-TRANS: no longer U6.B8
- net D14/RXI: no longer U6.A7
- net D14/RXI-TRANS: no longer U6.B7
- net D9/!SLEEP!: no longer U6.A3
- net D9/!SLEEP!-TRANS: no longer U6.B3
- net GND: now also S4.1, S4.4; no longer C17.2, C18.2, Q4.S, R5.1, S4.2, S4.6, U6.EPAD, U6.GND
- net VIN: now also Q2.S, S4.3, S4.6; no longer Q1.D, S4.4, S4.8
- net VIN_R3: now also D8.C; no longer Q2.D, S4.1, S4.5
Other:
- note removed: "3.3V (VCCA) -> 3.3V - 5V (VCCB)"
- note removed: "Bi-Directional Power Switch"
- note removed: "IOREF Selection"
- note removed: "USE ONLY IF THERE IS NO IOREF ON YOUR BASE BOARD"
- note removed: "XBee to R3 Footprint Level Translation"
- moved on the sheet: I2C_PU, J4, J5, J6, Q2, R14, R15
