File: Production/SparkFun_XBee_Arduino_Shield_Qwiic-Panel.brd (EAGLE design)
At the start: 120.9 x 213.4 mm, 1020 parts, among them J1 QWIIC_RIGHT_ANGLE, J13 QWIIC_RIGHT_ANGLE, J17 QWIIC_RIGHT_ANGLE, J21 QWIIC_RIGHT_ANGLE, J4 QWIIC_RIGHT_ANGLE, J9 QWIIC_RIGHT_ANGLE, Q1 220mA/50V/3.5Ω, Q11 3.1A/30V/105mΩ, Q12 220mA/50V/3.5Ω, Q13 20V/4.2A/52mΩ/1.4W, Q15 3.1A/30V/105mΩ, Q16 220mA/50V/3.5Ω, Q17 20V/4.2A/52mΩ/1.4W, Q19 3.1A/30V/105mΩ, Q2 20V/4.2A/52mΩ/1.4W, Q20 220mA/50V/3.5Ω, Q21 20V/4.2A/52mΩ/1.4W, Q23 3.1A/30V/105mΩ, Q24 220mA/50V/3.5Ω, Q3 3.1A/30V/105mΩ, Q5 20V/4.2A/52mΩ/1.4W, Q6 3.1A/30V/105mΩ, Q8 220mA/50V/3.5Ω, Q9 20V/4.2A/52mΩ/1.4W, U1 FSUSB42MUX, U10 FSUSB42MUX, U11 AP63203, U12 ESD Diode, U13 ESD Diode, U14 FT231XS, U15 FSUSB42MUX, U16 AP63203, U17 ESD Diode, U18 ESD Diode, U19 FT231XS, U2 AP63203, U20 FSUSB42MUX, U21 AP63203, U22 ESD Diode, U23 ESD Diode, U24 FT231XS, U25 FSUSB42MUX, U26 AP63203, U27 ESD Diode, U28 ESD Diode, U29 FT231XS, U3 ESD Diode, U30 FSUSB42MUX, U4 FT231XS, U5 ESD Diode, U6 AP63203, U7 ESD Diode, U8 ESD Diode, U9 FT231XS, X1 JUMPER-SMT_2_NO_SILK, X2 JUMPER-SMT_2_NO_SILK, X3 JUMPER-SMT_2_NO_SILK, X4 JUMPER-SMT_2_NO_SILK, X5 JUMPER-SMT_2_NO_SILK, X6 JUMPER-SMT_2_NO_SILK

Commit message: Adds new production file for v12
Parts:
- removed C61, C62, C75, C76: 10nF, SparkFun-Capacitors:0603
- removed C63, C65, C66, C69, C71, C77, C79, C80, C83: 0.1uF, SparkFun-Capacitors:0603
- removed C64, C78: 10uF, SparkFun-Capacitors:0603
- removed C67, C81: 47pF, SparkFun-Capacitors:0603
- removed C68, C82: 10pF, SparkFun-Capacitors:0603
- removed C70, C84: 4.7uF, SparkFun-Capacitors:0603
- removed C72, C73: 22uF, SparkFun-Capacitors:0603
- removed C74: 10uF, SparkFun-Capacitors:1210
- removed D37, D44, D45: 3A/10V/280mV, SparkFun-DiscreteSemi:SOD-323
- removed D38, D46: GREEN, SparkFun-LED:LED-0603
- removed D39, D40, D47, D48: 3A/40V/500mV, SparkFun-DiscreteSemi:SMA-DIODE
- removed D41: RED, SparkFun-LED:LED-0603
- removed D42: BLUE, SparkFun-LED:LED-0603
- removed D43: Yellow, SparkFun-LED:LED-0603
- removed DIRECT_USB, DIRECT_USB1, DIRECT_USB2, DIRECT_USB3, DIRECT_USB4, DIRECT_USB5: USB Female Type C Connector, SparkFun-Connectors:USB-C-16P-4LAYER-ISOLATED
- removed S25, S28, S29, S30: (no value), SparkFun-Switches:SWITCH_DPDT_SMD_AYZ0202
- removed S26, S27: (no value), SparkFun-Switches:TACTILE_SWITCH_SMD_5.2MM
- removed SHLD10, SHLD11, SHLD6, SHLD7, SHLD8, SHLD9: JUMPER-SMT_2_NC_TRACE_SILK, SparkFun-Jumpers:SMT-JUMPER_2_NC_TRACE_SILK
- removed U10, U15, U20, U25, U30: FSUSB42MUX, SparkFun-IC-Special-Function:MSOP10
- removed U11, U16, U21, U26: AP63203, SparkFun-IC-Power:SOT23-6
- removed U12, U13, U17, U18, U22, U23, U27, U28, U7, U8: ESD Diode, SparkFun-DiscreteSemi:SOT-23-6
- removed U14, U19, U24, U29, U9: FT231XS, SparkFun-IC-Comms:SSOP20_L
- added ARX, ARX1, ARX2, ARX3, ARX4, ARX5, ATX, ATX1, ATX2, ATX3, ATX4, ATX5: JUMPER-SMT_2_NC_TRACE_SILK, SparkFun-Jumpers:SMT-JUMPER_2_NC_TRACE_SILK
- added Q25, Q31: 20V/4.2A/52mΩ/1.4W, SparkFun-DiscreteSemi:SOT23-3
- added Q26, Q32: (no value), SparkFun-DiscreteSemi:SOT363_PHILIPS
- added Q27, Q33: 3.1A/30V/105mΩ, SparkFun-DiscreteSemi:SOT23-3
- added Q28, Q29, Q30, Q34, Q35, Q36: 220mA/50V/3.5Ω, SparkFun-DiscreteSemi:SOT23-3
- added U$571: (no value), prod:#XBEE_DIO0#62
- added U$572: (no value), prod:#XBEE_DIO9#62
- added U$573: (no value), prod:SOURCE54
- added U$574: (no value), prod:SHIELD55
- added U$575: (no value), prod:R3#R455
- added U$576: (no value), prod:USB#C58
- C12, C13, C23, C43, C52: value 0.1uF -> 22uF
- C14: value 4.7uF -> 10uF; device SparkFun-Capacitors:0603 -> SparkFun-Capacitors:1210
- C15, C35, C55: value 0.1uF -> 10nF
- C16, C45: value 22uF -> 10nF
- C17, C31: value 22uF -> 0.1uF
- C18: device SparkFun-Capacitors:1210 -> SparkFun-Capacitors:0603
- C19: value 10nF -> 47pF
- C20: value 10nF -> 10pF
- C22: value 10uF -> 22uF
- C24: value 0.1uF -> 10uF; device SparkFun-Capacitors:0603 -> SparkFun-Capacitors:1210
- C25: value 47pF -> 10nF
- C26: value 10pF -> 10nF
- C28: value 4.7uF -> 10uF
- C29, C49: value 0.1uF -> 47pF
- C30: value 22uF -> 10pF
- C32: value 10uF -> 22uF; device SparkFun-Capacitors:1210 -> SparkFun-Capacitors:0603
- C33: value 10nF -> 22uF
- C34: value 10nF -> 10uF; device SparkFun-Capacitors:0603 -> SparkFun-Capacitors:1210
- C36: value 10uF -> 10nF
- C38: value 0.1uF -> 10uF
- C42: value 4.7uF -> 22uF
- C44: value 22uF -> 10uF; device SparkFun-Capacitors:0603 -> SparkFun-Capacitors:1210
- C46: value 10uF -> 10nF; device SparkFun-Capacitors:1210 -> SparkFun-Capacitors:0603
- C47: value 10nF -> 0.1uF
- C48: value 10nF -> 10uF
- C50: value 10uF -> 10pF
- C53: value 47pF -> 22uF
- C54: value 10pF -> 10uF; device SparkFun-Capacitors:0603 -> SparkFun-Capacitors:1210
- C56: value 4.7uF -> 10nF
- C58: value 22uF -> 10uF
- C59: value 22uF -> 47pF
- C60: value 10uF -> 10pF; device SparkFun-Capacitors:1210 -> SparkFun-Capacitors:0603
- D1, D13: value 3A/10V/280mV -> RED; device SparkFun-DiscreteSemi:SOD-323 -> SparkFun-LED:LED-0603
- D10, D34: value BLUE -> GREEN
- D11, D35: value Yellow -> 3A/40V/500mV; device SparkFun-LED:LED-0603 -> SparkFun-DiscreteSemi:SMA-DIODE
- D12, D29, D36: value 3A/10V/280mV -> 3A/40V/500mV; device SparkFun-DiscreteSemi:SOD-323 -> SparkFun-DiscreteSemi:SMA-DIODE
- D14: value GREEN -> BLUE
- D15: value 3A/40V/500mV -> Yellow; device SparkFun-DiscreteSemi:SMA-DIODE -> SparkFun-LED:LED-0603
- D16: value 3A/40V/500mV -> GREEN; device SparkFun-DiscreteSemi:SMA-DIODE -> SparkFun-LED:LED-0603
- D17: value RED -> 3A/40V/500mV; device SparkFun-LED:LED-0603 -> SparkFun-DiscreteSemi:SMA-DIODE
- D18: value BLUE -> 3A/40V/500mV; device SparkFun-LED:LED-0603 -> SparkFun-DiscreteSemi:SMA-DIODE
- D19: value Yellow -> RED
- D20, D5: value 3A/10V/280mV -> BLUE; device SparkFun-DiscreteSemi:SOD-323 -> SparkFun-LED:LED-0603
- D21: value 3A/10V/280mV -> Yellow; device SparkFun-DiscreteSemi:SOD-323 -> SparkFun-LED:LED-0603
- D28: value 3A/10V/280mV -> GREEN; device SparkFun-DiscreteSemi:SOD-323 -> SparkFun-LED:LED-0603
- D30: value GREEN -> 3A/40V/500mV; device SparkFun-LED:LED-0603 -> SparkFun-DiscreteSemi:SMA-DIODE
- D31: value 3A/40V/500mV -> RED; device SparkFun-DiscreteSemi:SMA-DIODE -> SparkFun-LED:LED-0603
- D32: value 3A/40V/500mV -> BLUE; device SparkFun-DiscreteSemi:SMA-DIODE -> SparkFun-LED:LED-0603
- D33, D8: value RED -> Yellow
- Q10, Q18, Q22, Q4: value (none) -> 220mA/50V/3.5Ω; device SparkFun-DiscreteSemi:SOT363_PHILIPS -> SparkFun-DiscreteSemi:SOT23-3
- Q11, Q23: value 3.1A/30V/105mΩ -> 220mA/50V/3.5Ω
- Q17, Q2: value 20V/4.2A/52mΩ/1.4W -> 220mA/50V/3.5Ω
- Q19, Q6: value 3.1A/30V/105mΩ -> 20V/4.2A/52mΩ/1.4W
- Q20, Q8: value 220mA/50V/3.5Ω -> (none); device SparkFun-DiscreteSemi:SOT23-3 -> SparkFun-DiscreteSemi:SOT363_PHILIPS
- Q21, Q9: value 20V/4.2A/52mΩ/1.4W -> 3.1A/30V/105mΩ
- R1: value 100k -> 2.2k
- R13, R16: value 5.1k -> 2.2k
- R25, R40, R55, R70, R85: value 5.1k -> 1M
- R26, R41, R56, R71, R86: value 5.1k -> 330
- R27, R42, R57, R72, R87: value 100k -> 10k
- R28, R43, R58, R73, R88: value 1M -> 2.2k
- R29, R44, R59, R74, R89: value 330 -> 2.2k
- R30, R45, R60, R75, R90: value 10k -> 100k
- R9: value 2.2k -> 100k
- S10, S13, S14, S18, S3, S9: device SparkFun-Switches:SWITCH_DPDT_SMD_AYZ0202 -> SparkFun-Switches:TACTILE_SWITCH_SMD_5.2MM
- S11, S12, S16, S7: device SparkFun-Switches:TACTILE_SWITCH_SMD_5.2MM -> SparkFun-Switches:SWITCH_DPDT_SMD_AYZ0202
- U$100: device topmirror:#D1#AD1#8 -> SparkFun-Aesthetics:SFE_LOGO_FLAME_.2
- U$101: device topmirror:#D2#AD2#19 -> topmirror:#D1#AD1#8
- U$102: device topmirror:#D3#AD3#23 -> topmirror:#D2#AD2#19
- U$103: device topmirror:#D6##RTS##25 -> topmirror:#D3#AD3#23
- U$104: device topmirror:#D5#ASSOC#25 -> topmirror:#D6##RTS##25
- U$105: device topmirror:#D9##SLP##28 -> topmirror:#D5#ASSOC#25
- U$106: device topmirror:#D7##CTS##26 -> topmirror:#D9##SLP##28
- U$107: device topmirror:#D4#PICO#25 -> topmirror:#D7##CTS##26
- U$108: device topmirror:#D8##DTR##27 -> topmirror:#D4#PICO#25
- U$109: device topmirror:#RSSI#D10#17 -> topmirror:#D8##DTR##27
- U$110: device topmirror:#SDA#D11#9 -> topmirror:#RSSI#D10#17
- U$111: device topmirror:##RST##15 -> topmirror:#SDA#D11#9
- U$112: device topmirror:#POCI#D12#24 -> topmirror:##RST##15
- U$113: device topmirror:#RXI#D14#15 -> topmirror:#POCI#D12#24
- U$114: device topmirror:#TXO#D13#13 -> topmirror:#RXI#D14#15
- U$115: device topmirror:#EN#17 -> topmirror:#TXO#D13#13
- U$134: device topmirror:UART34 -> topmirror:#GND#0
- U$135, U$515, U$519: device topmirror:#GND#0 -> topmirror:#NC#1
- U$136: device topmirror:#NC#1 -> botmirror:#SDA#10
- U$137: device botmirror:#SDA#10 -> top:#SCL#7
- U$138, U$518: device top:#SCL#7 -> topmirror:#GND#0
- U$139, U$523: device topmirror:#GND#0 -> botmirror:#TXO#8
- U$140: device botmirror:#TXO#8 -> botmirror:#RXI#7
- U$141: device botmirror:#RXI#7 -> top:#3V3#1
- U$142, U$165, U$522: device top:#3V3#1 -> topmirror:#GND#0
- U$143: device topmirror:#GND#0 -> SparkFun-Aesthetics:SFE_LOGO_NAME_.2
- U$144: device SparkFun-Aesthetics:SFE_LOGO_NAME_.2 -> top:##SLP##28
- U$145: device top:##SLP##28 -> top:ASC32
- U$146: device topmirror:DIRECT_USB33 -> top:RSSI31
- U$147: device botmirror:#DUSB#31 -> top:PWR29
- U$148: device top:ASC32 -> topmirror:#GND#0
- U$149: device top:RSSI31 -> top:#3V3#1
- U$150: device top:PWR29 -> topmirror:#D0#AD0#18
- U$151: device topmirror:#SHLD1#37 -> top:ARDUINO1345
- U$152: device topmirror:#GND#0 -> top:XBEE340
- U$153: device top:#3V3#1 -> top:SHIELD1346
- U$154: device topmirror:#D0#AD0#18 -> topmirror:#5V#5
- U$155: device top:ARDUINO1345 -> topmirror:##DTR##27
- U$156: device top:XBEE340 -> top:##CTS##28
- U$157: device top:SHIELD1346 -> topmirror:#GND#0
- U$158: device topmirror:#5V#5 -> top:#3V3#1
- U$159: device topmirror:DEVELOPMENT1346 -> top:#PLED#20
- U$160: device topmirror:BOARD1347 -> pot:#IOLED#5
- U$161: device top:#I2C#13751 -> pot:IO49
- U$162: device topmirror:##DTR##27 -> top:VIN5
- U$163: device top:##CTS##28 -> bot:#PICO#27
- U$164: device topmirror:#GND#0 -> bot:#X1#10
- U$166, U$261: device pot:OFF311 -> topmirror:#GND#0
- U$167: device top:#PLED#20 -> topmirror:#5V#5
- U$168: device pot:#IOLED#5 -> top:#SDA#9
- U$169: device pot:IO49 -> bot:#SCL#13
- U$170, U$550: device top:VIN5 -> topmirror:#GND#0
- U$171: device bot:#PICO#27 -> botmirror:#EN#15
- U$172: device bot:#D9#6 -> top:#3V3#1
- U$173: device bot:#D0#3 -> botmirror:##RST##13
- U$174: device bot:#X1#10 -> topmirror:#VIN#4
- U$175: device bot:ON38 -> top:#UART#4048234
- U$176, U$272: device topmirror:#GND#0 -> prod:POWER49
- U$177, U$561: device topmirror:#GND#0 -> prod:DRX52
- U$178: device topmirror:#5V#5 -> prod:DTX53
- U$179: device top:#SDA#9 -> prod:DLINE45
- U$180: device bot:#SCL#13 -> prod:UART44
- U$181: device topmirror:#GND#0 -> prod:#DRX#56
- U$182: device botmirror:#EN#15 -> prod:#DTX#57
- U$183: device top:#3V3#1 -> prod:#TXO#61
- U$184: device botmirror:##RST##13 -> prod:#RXI#60
- U$185, U$565: device topmirror:#VIN#4 -> prod:#DRX#56
- U$186, U$566, U$89: device pot:#D0#3416 -> prod:#DTX#57
- U$187, U$90: device pot:#D9#3416 -> prod:#XBEE_DIO0#62
- U$188: device top:#UART#4048234 -> prod:#XBEE_DIO9#62
- U$189: device top:CONN4048235 -> prod:SOURCE54
- U$190: device top:OPEN4048238 -> prod:SHIELD55
- U$191: device top:#I2C#33 -> prod:R3#R455
- U$192: device bot:D03 -> prod:USB#C58
- U$193: device top:#RST#30 -> top:#I2C#33
- U$194: device SparkFun-Aesthetics:SFE_LOGO_FLAME_.2 -> bot:D03
- U$195: device topmirror:#D1#AD1#8 -> top:#RST#30
- U$196: device topmirror:#D2#AD2#19 -> SparkFun-Aesthetics:SFE_LOGO_FLAME_.2
- U$197: device topmirror:#D3#AD3#23 -> topmirror:#D1#AD1#8
- U$198: device topmirror:#D6##RTS##25 -> topmirror:#D2#AD2#19
- U$199: device topmirror:#D5#ASSOC#25 -> topmirror:#D3#AD3#23
- U$200: device topmirror:#D9##SLP##28 -> topmirror:#D6##RTS##25
- U$201: device topmirror:#D7##CTS##26 -> topmirror:#D5#ASSOC#25
- U$202: device topmirror:#D4#PICO#25 -> topmirror:#D9##SLP##28
- U$203: device topmirror:#D8##DTR##27 -> topmirror:#D7##CTS##26
- U$204: device topmirror:#RSSI#D10#17 -> topmirror:#D4#PICO#25
- U$205: device topmirror:#SDA#D11#9 -> topmirror:#D8##DTR##27
- U$206: device topmirror:##RST##15 -> topmirror:#RSSI#D10#17
- U$207: device topmirror:#POCI#D12#24 -> topmirror:#SDA#D11#9
- U$208: device topmirror:#RXI#D14#15 -> topmirror:##RST##15
- U$209: device topmirror:#TXO#D13#13 -> topmirror:#POCI#D12#24
- U$210: device topmirror:#EN#17 -> topmirror:#RXI#D14#15
- U$211: device topmirror:#ALED#21 -> topmirror:#TXO#D13#13
- U$212: device topmirror:#RLED#22 -> topmirror:#ALED#21
- U$213: device botmirror:#TXO#8 -> topmirror:#RLED#22
- U$214, U$331: device botmirror:#RXI#7 -> botmirror:#TXO#8
- U$215: device botmirror:#POCI#32 -> botmirror:#RXI#7
- U$216: device botmirror:##RST##13 -> botmirror:#POCI#32
- U$217: device topmirror:#RSSI#16 -> botmirror:##RST##13
- U$218: device botmirror:#SDA#10 -> topmirror:#RSSI#16
- U$219: device botmirror:#ASSOC#28 -> botmirror:#SDA#10
- U$220: device botmirror:##RTS##14 -> botmirror:#ASSOC#28
- U$221: device botmirror:##CS##26 -> botmirror:##RTS##14
- U$222: device botmirror:#SCLK#33 -> botmirror:##CS##26
- U$223: device botmirror:#SCL#9 -> botmirror:#SCLK#33
- U$224: device botmirror:#D0#3 -> botmirror:#SCL#9
- U$225: device topmirror:#SHLD#36 -> botmirror:#D0#3
- U$226: device topmirror:#NC#1 -> topmirror:#SHLD#36
- U$227, U$323: device botmirror:#NC#3 -> topmirror:#NC#1
- U$229, U$324: device topmirror:UART34 -> botmirror:#NC#3
- U$241: device topmirror:DIRECT_USB33 -> top:ASC32
- U$242: device botmirror:#DUSB#31 -> top:RSSI31
- U$243: device top:ASC32 -> top:PWR29
- U$244: device top:RSSI31 -> topmirror:#GND#0
- U$245: device top:PWR29 -> top:#3V3#1
- U$246: device topmirror:#SHLD1#37 -> topmirror:#D0#AD0#18
- U$247: device topmirror:#GND#0 -> top:ARDUINO1345
- U$248: device top:#3V3#1 -> top:XBEE340
- U$249: device topmirror:#D0#AD0#18 -> top:SHIELD1346
- U$250: device top:ARDUINO1345 -> topmirror:#5V#5
- U$251: device top:XBEE340 -> topmirror:##DTR##27
- U$252: device top:SHIELD1346 -> top:##CTS##28
- U$253: device topmirror:#5V#5 -> topmirror:#GND#0
- U$254: device topmirror:DEVELOPMENT1346 -> top:#3V3#1
- U$255: device topmirror:BOARD1347 -> top:#PLED#20
- U$256: device top:#I2C#13751 -> pot:#IOLED#5
- U$257: device topmirror:##DTR##27 -> pot:IO49
- U$258: device top:##CTS##28 -> top:VIN5
- U$259: device topmirror:#GND#0 -> bot:#PICO#27
- U$260: device top:#3V3#1 -> bot:#X1#10
- U$262, U$357: device top:#PLED#20 -> topmirror:#GND#0
- U$263: device pot:#IOLED#5 -> topmirror:#5V#5
- U$264: device pot:IO49 -> top:#SDA#9
- U$265: device top:VIN5 -> bot:#SCL#13
- U$266: device bot:#PICO#27 -> topmirror:#GND#0
- U$267: device bot:#D9#6 -> botmirror:#EN#15
- U$268: device bot:#D0#3 -> top:#3V3#1
- U$269: device bot:#X1#10 -> botmirror:##RST##13
- U$270: device bot:ON38 -> topmirror:#VIN#4
- U$271, U$367: device topmirror:#GND#0 -> top:#UART#4048234
- U$273: device topmirror:#5V#5 -> prod:DRX52
- U$274: device top:#SDA#9 -> prod:DTX53
- U$275: device bot:#SCL#13 -> prod:DLINE45
- U$276: device topmirror:#GND#0 -> prod:UART44
- U$277: device botmirror:#EN#15 -> prod:#DRX#56
- U$278: device top:#3V3#1 -> prod:#DTX#57
- U$279: device botmirror:##RST##13 -> prod:#TXO#61
- U$28: device topmirror:UART34 -> prod:DRX52
- U$280: device topmirror:#VIN#4 -> prod:#RXI#60
- U$281: device pot:#D0#3416 -> prod:#DRX#56
- U$282: device pot:#D9#3416 -> prod:#DTX#57
- U$283: device top:#UART#4048234 -> prod:#XBEE_DIO0#62
- U$284, U$92: device top:CONN4048235 -> prod:#XBEE_DIO9#62
- U$285, U$95: device top:OPEN4048238 -> prod:SOURCE54
- U$286: device top:#I2C#33 -> prod:SHIELD55
- U$287: device bot:D03 -> prod:R3#R455
- U$288: device top:#RST#30 -> prod:USB#C58
- U$289: device SparkFun-Aesthetics:SFE_LOGO_FLAME_.2 -> top:#I2C#33
- U$290: device topmirror:#D1#AD1#8 -> bot:D03
- U$291: device topmirror:#D2#AD2#19 -> top:#RST#30
- U$292: device topmirror:#D3#AD3#23 -> SparkFun-Aesthetics:SFE_LOGO_FLAME_.2
- U$293: device topmirror:#D6##RTS##25 -> topmirror:#D1#AD1#8
- U$294: device topmirror:#D5#ASSOC#25 -> topmirror:#D2#AD2#19
- U$295: device topmirror:#D9##SLP##28 -> topmirror:#D3#AD3#23
- U$296: device topmirror:#D7##CTS##26 -> topmirror:#D6##RTS##25
- U$297: device topmirror:#D4#PICO#25 -> topmirror:#D5#ASSOC#25
- U$298: device topmirror:#D8##DTR##27 -> topmirror:#D9##SLP##28
- U$299: device topmirror:#RSSI#D10#17 -> topmirror:#D7##CTS##26
- U$300: device topmirror:#SDA#D11#9 -> topmirror:#D4#PICO#25
- U$301: device topmirror:##RST##15 -> topmirror:#D8##DTR##27
- U$302: device topmirror:#POCI#D12#24 -> topmirror:#RSSI#D10#17
- U$303: device topmirror:#RXI#D14#15 -> topmirror:#SDA#D11#9
- U$304: device topmirror:#TXO#D13#13 -> topmirror:##RST##15
- U$305: device topmirror:#EN#17 -> topmirror:#POCI#D12#24
- U$306: device topmirror:#ALED#21 -> topmirror:#RXI#D14#15
- U$307: device topmirror:#RLED#22 -> topmirror:#TXO#D13#13
- U$308: device botmirror:#TXO#8 -> topmirror:#ALED#21
- U$309: device botmirror:#RXI#7 -> topmirror:#RLED#22
- U$310: device botmirror:#POCI#32 -> botmirror:#TXO#8
- U$311: device botmirror:##RST##13 -> botmirror:#RXI#7
- U$312: device topmirror:#RSSI#16 -> botmirror:#POCI#32
- U$313: device botmirror:#SDA#10 -> botmirror:##RST##13
- U$314: device botmirror:#ASSOC#28 -> topmirror:#RSSI#16
- U$315: device botmirror:##RTS##14 -> botmirror:#SDA#10
- U$316: device botmirror:##CS##26 -> botmirror:#ASSOC#28
- U$317: device botmirror:#SCLK#33 -> botmirror:##RTS##14
- U$318: device botmirror:#SCL#9 -> botmirror:##CS##26
- U$319: device botmirror:#D0#3 -> botmirror:#SCLK#33
- U$320: device topmirror:#SHLD#36 -> botmirror:#SCL#9
- U$321: device topmirror:#NC#1 -> botmirror:#D0#3
- U$322, U$418: device botmirror:#NC#3 -> topmirror:#SHLD#36
- U$325, U$420: device topmirror:#GND#0 -> botmirror:#NC#3
- U$326: device topmirror:#NC#1 -> topmirror:#GND#0
- U$327: device botmirror:#SDA#10 -> topmirror:#NC#1
- U$328: device top:#SCL#7 -> botmirror:#SDA#10
- U$329: device topmirror:#GND#0 -> top:#SCL#7
- U$330: device botmirror:#TXO#8 -> topmirror:#GND#0
- U$332: device top:#3V3#1 -> botmirror:#RXI#7
- U$333, U$437, U$556: device topmirror:#GND#0 -> top:#3V3#1
- U$334: device SparkFun-Aesthetics:SFE_LOGO_NAME_.2 -> topmirror:#GND#0
- U$335: device top:##SLP##28 -> SparkFun-Aesthetics:SFE_LOGO_NAME_.2
- U$336: device topmirror:DIRECT_USB33 -> top:##SLP##28
- U$337: device botmirror:#DUSB#31 -> top:ASC32
- U$338: device top:ASC32 -> top:RSSI31
- U$339: device top:RSSI31 -> top:PWR29
- U$34: device bot:#D9#6 -> prod:DTX53
- U$340: device top:PWR29 -> topmirror:#GND#0
- U$341: device topmirror:#SHLD1#37 -> top:#3V3#1
- U$342: device topmirror:#GND#0 -> topmirror:#D0#AD0#18
- U$343: device top:#3V3#1 -> top:ARDUINO1345
- U$344: device topmirror:#D0#AD0#18 -> top:XBEE340
- U$345: device top:ARDUINO1345 -> top:SHIELD1346
- U$346: device top:XBEE340 -> topmirror:#5V#5
- U$347: device top:SHIELD1346 -> topmirror:##DTR##27
- U$348: device topmirror:#5V#5 -> top:##CTS##28
- U$349: device topmirror:DEVELOPMENT1346 -> topmirror:#GND#0
- U$350: device topmirror:BOARD1347 -> top:#3V3#1
- U$351: device top:#I2C#13751 -> top:#PLED#20
- U$352: device topmirror:##DTR##27 -> pot:#IOLED#5
- U$353: device top:##CTS##28 -> pot:IO49
- U$354: device topmirror:#GND#0 -> top:VIN5
- U$355: device top:#3V3#1 -> bot:#PICO#27
- U$356: device pot:OFF311 -> bot:#X1#10
- U$358, U$453: device pot:#IOLED#5 -> topmirror:#GND#0
- U$359: device pot:IO49 -> topmirror:#5V#5
- U$360: device top:VIN5 -> top:#SDA#9
- U$361: device bot:#PICO#27 -> bot:#SCL#13
- U$362: device bot:#D9#6 -> topmirror:#GND#0
- U$363: device bot:#D0#3 -> botmirror:#EN#15
- U$364: device bot:#X1#10 -> top:#3V3#1
- U$365: device bot:ON38 -> botmirror:##RST##13
- U$366, U$462: device topmirror:#GND#0 -> topmirror:#VIN#4
- U$368: device topmirror:#5V#5 -> prod:POWER49
- U$369: device top:#SDA#9 -> prod:DRX52
- U$370: device bot:#SCL#13 -> prod:DTX53
- U$371: device topmirror:#GND#0 -> prod:DLINE45
- U$372: device botmirror:#EN#15 -> prod:UART44
- U$373: device top:#3V3#1 -> prod:#DRX#56
- U$374: device botmirror:##RST##13 -> prod:#DTX#57
- U$375: device topmirror:#VIN#4 -> prod:#TXO#61
- U$376: device pot:#D0#3416 -> prod:#RXI#60
- U$377: device pot:#D9#3416 -> prod:#DRX#56
- U$378: device top:#UART#4048234 -> prod:#DTX#57
- U$379: device top:CONN4048235 -> prod:#XBEE_DIO0#62
- U$380: device top:OPEN4048238 -> prod:#XBEE_DIO9#62
- U$381: device top:#I2C#33 -> prod:SOURCE54
- U$382: device bot:D03 -> prod:SHIELD55
- U$383: device top:#RST#30 -> prod:R3#R455
- U$384: device SparkFun-Aesthetics:SFE_LOGO_FLAME_.2 -> prod:USB#C58
- U$385: device topmirror:#D1#AD1#8 -> top:#I2C#33
- U$386: device topmirror:#D2#AD2#19 -> bot:D03
- U$387: device topmirror:#D3#AD3#23 -> top:#RST#30
- U$388: device topmirror:#D6##RTS##25 -> SparkFun-Aesthetics:SFE_LOGO_FLAME_.2
- U$389: device topmirror:#D5#ASSOC#25 -> topmirror:#D1#AD1#8
- U$390: device topmirror:#D9##SLP##28 -> topmirror:#D2#AD2#19
- U$391: device topmirror:#D7##CTS##26 -> topmirror:#D3#AD3#23
- U$392: device topmirror:#D4#PICO#25 -> topmirror:#D6##RTS##25
- U$393: device topmirror:#D8##DTR##27 -> topmirror:#D5#ASSOC#25
- U$394: device topmirror:#RSSI#D10#17 -> topmirror:#D9##SLP##28
- U$395: device topmirror:#SDA#D11#9 -> topmirror:#D7##CTS##26
- U$396: device topmirror:##RST##15 -> topmirror:#D4#PICO#25
- U$397: device topmirror:#POCI#D12#24 -> topmirror:#D8##DTR##27
- U$398: device topmirror:#RXI#D14#15 -> topmirror:#RSSI#D10#17
- U$399: device topmirror:#TXO#D13#13 -> topmirror:#SDA#D11#9
- U$400: device topmirror:#EN#17 -> topmirror:##RST##15
- U$401: device topmirror:#ALED#21 -> topmirror:#POCI#D12#24
- U$402: device topmirror:#RLED#22 -> topmirror:#RXI#D14#15
- U$403: device botmirror:#TXO#8 -> topmirror:#TXO#D13#13
- U$404: device botmirror:#RXI#7 -> topmirror:#ALED#21
- U$405: device botmirror:#POCI#32 -> topmirror:#RLED#22
- U$406: device botmirror:##RST##13 -> botmirror:#TXO#8
- U$407: device topmirror:#RSSI#16 -> botmirror:#RXI#7
- U$408: device botmirror:#SDA#10 -> botmirror:#POCI#32
- U$409: device botmirror:#ASSOC#28 -> botmirror:##RST##13
- U$410: device botmirror:##RTS##14 -> topmirror:#RSSI#16
- U$411: device botmirror:##CS##26 -> botmirror:#SDA#10
- U$412: device botmirror:#SCLK#33 -> botmirror:#ASSOC#28
- U$413: device botmirror:#SCL#9 -> botmirror:##RTS##14
- U$414: device botmirror:#D0#3 -> botmirror:##CS##26
- U$415: device topmirror:#SHLD#36 -> botmirror:#SCLK#33
- U$416: device topmirror:#NC#1 -> botmirror:#SCL#9
- U$417, U$513: device botmirror:#NC#3 -> botmirror:#D0#3
- U$419: device topmirror:UART34 -> topmirror:#NC#1
- U$42: device bot:#D0#3 -> prod:DLINE45
- U$421, U$516: device topmirror:#NC#1 -> botmirror:#NC#3
- U$422: device botmirror:#SDA#10 -> topmirror:#GND#0
- U$423: device top:#SCL#7 -> topmirror:#NC#1
- U$424: device topmirror:#GND#0 -> botmirror:#SDA#10
- U$425: device botmirror:#TXO#8 -> top:#SCL#7
- U$426: device botmirror:#RXI#7 -> topmirror:#GND#0
- U$427: device top:#3V3#1 -> botmirror:#TXO#8
- U$428: device topmirror:#GND#0 -> botmirror:#RXI#7
- U$429: device SparkFun-Aesthetics:SFE_LOGO_NAME_.2 -> top:#3V3#1
- U$430: device top:##SLP##28 -> topmirror:#GND#0
- U$431: device topmirror:DIRECT_USB33 -> SparkFun-Aesthetics:SFE_LOGO_NAME_.2
- U$432: device botmirror:#DUSB#31 -> top:##SLP##28
- U$436: device topmirror:#SHLD1#37 -> topmirror:#GND#0
- U$438: device top:#3V3#1 -> topmirror:#D0#AD0#18
- U$439: device topmirror:#D0#AD0#18 -> top:ARDUINO1345
- U$440: device top:ARDUINO1345 -> top:XBEE340
- U$441: device top:XBEE340 -> top:SHIELD1346
- U$442: device top:SHIELD1346 -> topmirror:#5V#5
- U$443: device topmirror:#5V#5 -> topmirror:##DTR##27
- U$444: device topmirror:DEVELOPMENT1346 -> top:##CTS##28
- U$445: device topmirror:BOARD1347 -> topmirror:#GND#0
- U$446: device top:#I2C#13751 -> top:#3V3#1
- U$447: device topmirror:##DTR##27 -> top:#PLED#20
- U$448: device top:##CTS##28 -> pot:#IOLED#5
- U$449: device topmirror:#GND#0 -> pot:IO49
- U$450: device top:#3V3#1 -> top:VIN5
- U$451: device pot:OFF311 -> bot:#PICO#27
- U$452: device top:#PLED#20 -> bot:#X1#10
- U$454, U$549: device pot:IO49 -> topmirror:#GND#0
- U$455: device top:VIN5 -> topmirror:#5V#5
- U$456: device bot:#PICO#27 -> top:#SDA#9
- U$457: device bot:#D9#6 -> bot:#SCL#13
- U$458: device bot:#D0#3 -> topmirror:#GND#0
- U$459: device bot:#X1#10 -> botmirror:#EN#15
- U$46: device bot:ON38 -> prod:SHIELD55
- U$460: device bot:ON38 -> top:#3V3#1
- U$461, U$557: device topmirror:#GND#0 -> botmirror:##RST##13
- U$463: device topmirror:#5V#5 -> top:#UART#4048234
- U$464: device top:#SDA#9 -> prod:POWER49
- U$465: device bot:#SCL#13 -> prod:DRX52
- U$466: device topmirror:#GND#0 -> prod:DTX53
- U$467: device botmirror:#EN#15 -> prod:DLINE45
- U$468: device top:#3V3#1 -> prod:UART44
- U$469: device botmirror:##RST##13 -> prod:#DRX#56
- U$470: device topmirror:#VIN#4 -> prod:#DTX#57
- U$471: device pot:#D0#3416 -> prod:#TXO#61
- U$472: device pot:#D9#3416 -> prod:#RXI#60
- U$473: device top:#UART#4048234 -> prod:#DRX#56
- U$474: device top:CONN4048235 -> prod:#DTX#57
- U$475: device top:OPEN4048238 -> prod:#XBEE_DIO0#62
- U$476: device top:#I2C#33 -> prod:#XBEE_DIO9#62
- U$477: device bot:D03 -> prod:SOURCE54
- U$478: device top:#RST#30 -> prod:SHIELD55
- U$479: device SparkFun-Aesthetics:SFE_LOGO_FLAME_.2 -> prod:R3#R455
- U$48: device topmirror:#EN#17 -> prod:UART44
- U$480: device topmirror:#D1#AD1#8 -> prod:USB#C58
- U$481: device topmirror:#D2#AD2#19 -> top:#I2C#33
- U$482: device topmirror:#D3#AD3#23 -> bot:D03
- U$483: device topmirror:#D6##RTS##25 -> top:#RST#30
- U$484: device topmirror:#D5#ASSOC#25 -> SparkFun-Aesthetics:SFE_LOGO_FLAME_.2
- U$485: device topmirror:#D9##SLP##28 -> topmirror:#D1#AD1#8
- U$486: device topmirror:#D7##CTS##26 -> topmirror:#D2#AD2#19
- U$487: device topmirror:#D4#PICO#25 -> topmirror:#D3#AD3#23
- U$488: device topmirror:#D8##DTR##27 -> topmirror:#D6##RTS##25
- U$489: device topmirror:#RSSI#D10#17 -> topmirror:#D5#ASSOC#25
- U$490: device topmirror:#SDA#D11#9 -> topmirror:#D9##SLP##28
- U$491: device topmirror:##RST##15 -> topmirror:#D7##CTS##26
- U$492: device topmirror:#POCI#D12#24 -> topmirror:#D4#PICO#25
- U$493: device topmirror:#RXI#D14#15 -> topmirror:#D8##DTR##27
- U$494: device topmirror:#TXO#D13#13 -> topmirror:#RSSI#D10#17
- U$495: device topmirror:#EN#17 -> topmirror:#SDA#D11#9
- U$496: device topmirror:#ALED#21 -> topmirror:##RST##15
- U$497: device topmirror:#RLED#22 -> topmirror:#POCI#D12#24
- U$498: device botmirror:#TXO#8 -> topmirror:#RXI#D14#15
- U$499: device botmirror:#RXI#7 -> topmirror:#TXO#D13#13
- U$500: device botmirror:#POCI#32 -> topmirror:#ALED#21
- U$501: device botmirror:##RST##13 -> topmirror:#RLED#22
- U$502: device topmirror:#RSSI#16 -> botmirror:#TXO#8
- U$503: device botmirror:#SDA#10 -> botmirror:#RXI#7
- U$504: device botmirror:#ASSOC#28 -> botmirror:#POCI#32
- U$505: device botmirror:##RTS##14 -> botmirror:##RST##13
- U$506: device botmirror:##CS##26 -> topmirror:#RSSI#16
- U$507: device botmirror:#SCLK#33 -> botmirror:#SDA#10
- U$508: device botmirror:#SCL#9 -> botmirror:#ASSOC#28
- U$509: device botmirror:#D0#3 -> botmirror:##RTS##14
- U$510: device topmirror:#SHLD#36 -> botmirror:##CS##26
- U$511: device topmirror:#NC#1 -> botmirror:#SCLK#33
- U$512: device botmirror:#NC#3 -> botmirror:#SCL#9
- U$514: device topmirror:UART34 -> topmirror:#SHLD#36
- U$517: device botmirror:#SDA#10 -> botmirror:#NC#3
- U$520: device botmirror:#TXO#8 -> botmirror:#SDA#10
- U$521: device botmirror:#RXI#7 -> top:#SCL#7
- U$524: device SparkFun-Aesthetics:SFE_LOGO_NAME_.2 -> botmirror:#RXI#7
- U$525: device top:##SLP##28 -> top:#3V3#1
- U$526: device topmirror:DIRECT_USB33 -> topmirror:#GND#0
- U$527: device botmirror:#DUSB#31 -> SparkFun-Aesthetics:SFE_LOGO_NAME_.2
- U$528: device top:ASC32 -> top:##SLP##28
- U$529: device top:RSSI31 -> top:ASC32
- U$530: device top:PWR29 -> top:RSSI31
- U$531: device topmirror:#SHLD1#37 -> top:PWR29
- U$539: device topmirror:DEVELOPMENT1346 -> topmirror:##DTR##27
- U$540: device topmirror:BOARD1347 -> top:##CTS##28
- U$541: device top:#I2C#13751 -> topmirror:#GND#0
- U$542: device topmirror:##DTR##27 -> top:#3V3#1
- U$543: device top:##CTS##28 -> top:#PLED#20
- U$544: device topmirror:#GND#0 -> pot:#IOLED#5
- U$545: device top:#3V3#1 -> pot:IO49
- U$546: device pot:OFF311 -> top:VIN5
- U$547: device top:#PLED#20 -> bot:#PICO#27
- U$548: device pot:#IOLED#5 -> bot:#X1#10
- U$551: device bot:#PICO#27 -> topmirror:#5V#5
- U$552: device bot:#D9#6 -> top:#SDA#9
- U$553: device bot:#D0#3 -> bot:#SCL#13
- U$554: device bot:#X1#10 -> topmirror:#GND#0
- U$555: device bot:ON38 -> botmirror:#EN#15
- U$558: device topmirror:#5V#5 -> topmirror:#VIN#4
- U$559: device top:#SDA#9 -> top:#UART#4048234
- U$560: device bot:#SCL#13 -> prod:POWER49
- U$562: device botmirror:#EN#15 -> prod:DTX53
- U$563: device top:#3V3#1 -> prod:DLINE45
- U$564: device botmirror:##RST##13 -> prod:UART44
- U$567: device pot:#D9#3416 -> prod:#TXO#61
- U$568: device top:#UART#4048234 -> prod:#RXI#60
- U$569: device top:CONN4048235 -> prod:#DRX#56
- U$570: device top:OPEN4048238 -> prod:#DTX#57
- U$69: device pot:OFF311 -> prod:R3#R455
- U$71: device topmirror:DIRECT_USB33 -> prod:#DRX#56
- U$72: device botmirror:#DUSB#31 -> prod:#DTX#57
- U$73: device top:#I2C#13751 -> prod:#TXO#61
- U$75: device topmirror:#SHLD1#37 -> prod:POWER49
- U$85: device topmirror:DEVELOPMENT1346 -> prod:#RXI#60
- U$86: device topmirror:BOARD1347 -> prod:#DRX#56
- U$96: device top:#I2C#33 -> prod:USB#C58
- U$97: device bot:D03 -> top:#I2C#33
- U$98: device top:#RST#30 -> bot:D03
- U$99: device SparkFun-Aesthetics:SFE_LOGO_FLAME_.2 -> top:#RST#30
- U1: value FSUSB42MUX -> AP63203; device SparkFun-IC-Special-Function:MSOP10 -> SparkFun-IC-Power:SOT23-6
- U3, U5: value ESD Diode -> AP63203; device SparkFun-DiscreteSemi:SOT-23-6 -> SparkFun-IC-Power:SOT23-6
- U4: value FT231XS -> AP63203; device SparkFun-IC-Comms:SSOP20_L -> SparkFun-IC-Power:SOT23-6
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Connections:
- removed net 3.3V_SW: B1.3.3V, Q3.2, S5.3, S5.6
- removed net 3.3V_SW1: B2.3.3V, Q6.2, S9.3, S9.6
- removed net 3.3V_SW2: B3.3.3V, Q11.2, S14.3, S14.6
- removed net 3.3V_SW3: B4.3.3V, Q15.2, S19.3, S19.6
- removed net 3.3V_SW4: B5.3.3V, Q19.2, S24.3, S24.6
- removed net 3.3V_SW5: B6.3.3V, Q23.2, S29.3, S29.6
- removed net D+: U4.11, U5.6, UART.A6, UART.B6
- removed net D+1: U7.6, U9.11, UART1.A6, UART1.B6
- removed net D+2: U12.6, U14.11, UART2.A6, UART2.B6
- removed net D+3: U17.6, U19.11, UART3.A6, UART3.B6
- removed net D+4: U22.6, U24.11, UART4.A6, UART4.B6
- removed net D+5: U27.6, U29.11, UART5.A6, UART5.B6
- removed net D-: U4.12, U5.4, UART.A7, UART.B7
- removed net D-1: U7.4, U9.12, UART1.A7, UART1.B7
- removed net D-2: U12.4, U14.12, UART2.A7, UART2.B7
- removed net D-3: U17.4, U19.12, UART3.A7, UART3.B7
- removed net D-4: U22.4, U24.12, UART4.A7, UART4.B7
- removed net D-5: U27.4, U29.12, UART5.A7, UART5.B7
- removed net DIRECT_D+: DIRECT_USB.A6, DIRECT_USB.B6, U1.9, U3.6
- removed net DIRECT_D+1: DIRECT_USB1.A6, DIRECT_USB1.B6, U10.9, U8.6
- removed net DIRECT_D+2: DIRECT_USB2.A6, DIRECT_USB2.B6, U13.6, U15.9
- removed net DIRECT_D+3: DIRECT_USB3.A6, DIRECT_USB3.B6, U18.6, U20.9
- removed net DIRECT_D+4: DIRECT_USB4.A6, DIRECT_USB4.B6, U23.6, U25.9
- removed net DIRECT_D+5: DIRECT_USB5.A6, DIRECT_USB5.B6, U28.6, U30.9
- removed net DIRECT_D-: DIRECT_USB.A7, DIRECT_USB.B7, U1.8, U3.4
- removed net DIRECT_D-1: DIRECT_USB1.A7, DIRECT_USB1.B7, U10.8, U8.4
- removed net DIRECT_D-2: DIRECT_USB2.A7, DIRECT_USB2.B7, U13.4, U15.8
- removed net DIRECT_D-3: DIRECT_USB3.A7, DIRECT_USB3.B7, U18.4, U20.8
- removed net DIRECT_D-4: DIRECT_USB4.A7, DIRECT_USB4.B7, U23.4, U25.8
- removed net DIRECT_D-5: DIRECT_USB5.A7, DIRECT_USB5.B7, U28.4, U30.8
- removed net DIRECT_SELECT: S3.2, S3.5, U1.2
- removed net DIRECT_SELECT1: S8.2, S8.5, U10.2
- removed net DIRECT_SELECT2: S13.2, S13.5, U15.2
- removed net DIRECT_SELECT3: S18.2, S18.5, U20.2
- removed net DIRECT_SELECT4: S23.2, S23.5, U25.2
- removed net DIRECT_SELECT5: S28.2, S28.5, U30.2
- removed net DIRECT_USB: R1.2, S3.1, S3.4
- removed net DIRECT_USB1: R24.2, S8.1, S8.4
- removed net DIRECT_USB2: R39.2, S13.1, S13.4
- removed net DIRECT_USB3: R54.2, S18.1, S18.4
- removed net DIRECT_USB4: R69.2, S23.1, S23.4
- removed net DIRECT_USB5: R84.2, S28.1, S28.4
- removed net N$105 (its old number): D40.A, X5.2
- removed net N$106 (its old number): I2C_PU5.3, R76.2
- removed net N$115: D43.C, RLED5.2
- removed net N$118: DIRECT_USB5.B5, R86.2
- removed net N$119: DIRECT_USB5.A5, R85.2
- removed net N$120: Q22.2, Q22.5, Q22.6, R87.2
- removed net N$121: Q21.1, Q22.3, R88.2
- removed net N$122: D46.A, R89.2
- removed net N$123: D46.C, IO6.2
- removed net N$124: Q23.1, S29.2, S29.5
- removed net N$125: D47.A, Q23.3
- removed net N$126: D48.A, X6.2
- removed net N$29 (its old number): C15.2, L2.P$1, U6.5
- removed net N$30 (its old number): D11.A, R21.2
- removed net N$48 (its old number): D17.C, PLED2.2
- removed net N$49 (its old number): C29.1, U11.6
- removed net N$67 (its old number): D26.A, R49.2
- removed net N$68 (its old number): ALED3.2, D26.C
- removed net N$86 (its old number): I2C_PU4.1, R62.2
- removed net N$87 (its old number): D33.A, R63.2
- removed net SHLD10: SHLD10.2, UART5.SHLD1, UART5.SHLD2, UART5.SHLD3, UART5.SHLD4, UART5.SHLD5, UART5.SHLD6, UART5.SHLD7, UART5.SHLD8
- removed net SHLD11: DIRECT_USB5.SHLD1, DIRECT_USB5.SHLD2, DIRECT_USB5.SHLD3, DIRECT_USB5.SHLD4, DIRECT_USB5.SHLD5, DIRECT_USB5.SHLD6, DIRECT_USB5.SHLD7, DIRECT_USB5.SHLD8, SHLD11.2
- removed net SHLD6: SHLD6.2, UART3.SHLD1, UART3.SHLD2, UART3.SHLD3, UART3.SHLD4, UART3.SHLD5, UART3.SHLD6, UART3.SHLD7, UART3.SHLD8
- removed net SHLD7: DIRECT_USB3.SHLD1, DIRECT_USB3.SHLD2, DIRECT_USB3.SHLD3, DIRECT_USB3.SHLD4, DIRECT_USB3.SHLD5, DIRECT_USB3.SHLD6, DIRECT_USB3.SHLD7, DIRECT_USB3.SHLD8, SHLD7.2
- removed net SHLD8: SHLD8.2, UART4.SHLD1, UART4.SHLD2, UART4.SHLD3, UART4.SHLD4, UART4.SHLD5, UART4.SHLD6, UART4.SHLD7, UART4.SHLD8
- removed net SHLD9: DIRECT_USB4.SHLD1, DIRECT_USB4.SHLD2, DIRECT_USB4.SHLD3, DIRECT_USB4.SHLD4, DIRECT_USB4.SHLD5, DIRECT_USB4.SHLD6, DIRECT_USB4.SHLD7, DIRECT_USB4.SHLD8, SHLD9.2
- removed net VCC: C1.1, D1.C, D5.C, R3.2, U2.3, X1.1
- removed net VCC1: C18.1, D12.C, D13.C, R20.2, U6.3, X2.1
- removed net VCC2: C32.1, D20.C, D21.C, R35.2, U11.3, X3.1
- removed net VCC3: C46.1, D28.C, D29.C, R50.2, U16.3, X4.1
- removed net VCC4: C60.1, D36.C, D37.C, R65.2, U21.3, X5.1
- removed net VCC5: C74.1, D44.C, D45.C, R80.2, U26.3, X6.1
- removed net V_USB_1: D12.A, DIRECT_USB1.VBUS1, DIRECT_USB1.VBUS2, U8.5
- removed net V_USB_2: D1.A, DIRECT_USB.VBUS1, DIRECT_USB.VBUS2, U3.5
- removed net V_USB_3: D20.A, DIRECT_USB2.VBUS1, DIRECT_USB2.VBUS2, U13.5
- removed net V_USB_4: D28.A, DIRECT_USB3.VBUS1, DIRECT_USB3.VBUS2, U18.5
- removed net V_USB_5: D36.A, DIRECT_USB4.VBUS1, DIRECT_USB4.VBUS2, U23.5
- removed net V_USB_6: D44.A, DIRECT_USB5.VBUS1, DIRECT_USB5.VBUS2, U28.5
- removed net XBEE_D+/SDA: J2.7, U1.3
- removed net XBEE_D+/SDA1: J8.7, U10.3
- removed net XBEE_D+/SDA2: J12.7, U15.3
- removed net XBEE_D+/SDA3: J16.7, U20.3
- removed net XBEE_D+/SDA4: J20.7, U25.3
- removed net XBEE_D+/SDA5: J24.7, U30.3
- removed net XBEE_D-: J2.8, U1.4
- removed net XBEE_D-1: J8.8, U10.4
- removed net XBEE_D-2: J12.8, U15.4
- removed net XBEE_D-3: J16.8, U20.4
- removed net XBEE_D-4: J20.8, U25.4
- removed net XBEE_D-5: J24.8, U30.4
- new net 3.3V_R1: B2.3.3V, Q9.2, R27.2, R28.2, R29.2, S7.3, S7.6
- new net 3.3V_R2: B3.3.3V, Q15.2, R42.2, R43.2, R44.2, S11.3, S11.6
- new net 3.3V_R3: B1.3.3V, Q3.2, R1.2, R4.2, R5.2, S5.3, S5.6
- new net 3.3V_R4: B4.3.3V, Q21.2, R57.2, R58.2, R59.2, S15.3, S15.6
- new net 3.3V_R5: B5.3.3V, Q27.2, R72.2, R73.2, R74.2, S19.3, S19.6
- new net 3.3V_R6: B6.3.3V, Q33.2, R87.2, R88.2, R89.2, S23.3, S23.6
- new net D_RX: ARX.2, B1.D2
- new net D_RX1: ARX1.2, B2.D2
- new net D_RX2: ARX2.2, B3.D2
- new net D_RX3: ARX3.2, B4.D2
- new net D_RX4: ARX4.2, B5.D2
- new net D_RX5: ARX5.2, B6.D2
- new net D_RX_JUMP: ARX.1, S4.4
- new net D_RX_JUMP1: ARX1.1, S8.4
- new net D_RX_JUMP2: ARX2.1, S12.4
- new net D_RX_JUMP3: ARX3.1, S16.4
- new net D_RX_JUMP4: ARX4.1, S20.4
- new net D_RX_JUMP5: ARX5.1, S24.4
- new net D_TX: ATX.2, B1.D3
- new net D_TX1: ATX1.2, B2.D3
- new net D_TX2: ATX2.2, B3.D3
- new net D_TX3: ATX3.2, B4.D3
- new net D_TX4: ATX4.2, B5.D3
- new net D_TX5: ATX5.2, B6.D3
- new net D_TX_JUMP: ATX.1, S4.1
- new net D_TX_JUMP1: ATX1.1, S8.1
- new net D_TX_JUMP2: ATX2.1, S12.1
- new net D_TX_JUMP3: ATX3.1, S16.1
- new net D_TX_JUMP4: ATX4.1, S20.1
- new net D_TX_JUMP5: ATX5.1, S24.1
- new net N$32: Q6.1, Q8.3, R25.2
- new net N$33: D10.A, R26.2
- new net N$53: D16.C, IO2.2
- new net N$54: Q15.1, S11.2, S11.5
- new net N$74: D23.A, Q21.3, R60.2
- new net N$75: D24.A, X4.2
- new net N$95: I2C_PU4.1, Q30.1, R62.2
- new net N$96: I2C_PU5.3, Q35.1, R76.2
- new net R3_D1/SCL: B1.SCL, Q4.3, R4.1
- new net R3_D1/SCL1: B2.SCL, Q12.3, R29.1
- new net R3_D1/SCL2: B3.SCL, Q18.3, R44.1
- new net R3_D1/SCL3: B4.SCL, Q24.3, R59.1
- new net R3_D1/SCL4: B5.SCL, Q30.3, R74.1
- new net R3_D1/SCL5: B6.SCL, Q36.3, R89.1
- new net R3_D11/SDA: B1.SDA, Q2.3, R1.1
- new net R3_D11/SDA1: B2.SDA, Q11.3, R28.1
- new net R3_D11/SDA2: B3.SDA, Q17.3, R43.1
- new net R3_D11/SDA3: B4.SDA, Q23.3, R58.1
- new net R3_D11/SDA4: B5.SDA, Q29.3, R73.1
- new net R3_D11/SDA5: B6.SDA, Q35.3, R88.1
- net !RESET!1: now also C15.1, S3.1, S3.2; no longer C19.1, S6.1, S6.2
- net !RESET!2: now also C25.1, S9.1, S9.2; no longer C33.1, S11.1, S11.2
- net !RESET!3: now also C35.1, S13.1, S13.2; no longer C47.1, S16.1, S16.2
- net !RESET!4: now also C45.1, S17.1, S17.2; no longer C61.1, S21.1, S21.2
- net !RESET!5: now also C55.1, S21.1, S21.2; no longer C75.1, S26.1, S26.2
- net 3.3V: no longer C11.1, C12.1, C13.1, C14.1, Q1.1, R1.1, R5.2, U1.1, U4.13, U4.14, U4.15, U4.3
- net 3.3V1: now also C16.1, C17.1, C18.1, C19.1, D11.C, Q6.2, Q8.4; no longer C21.1, C22.1, C23.1, C24.1, C25.1, C26.1, C27.1, C28.1, D15.C, Q2.2, Q4.4, Q8.1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
- net 3.3V2: now also C26.1, C27.1, C28.1, C29.1, C30.1, D17.C, Q13.2, Q14.4; no longer C34.1, C35.1, C36.1, C37.1, C38.1, C39.1, C40.1, C41.1, C42.1, D23.C, Q10.4, Q12.1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
- net 3.3V3: now also C36.1, C37.1, C38.1, C39.1, C40.1, D23.C, Q19.2, Q20.4; no longer C48.1, C49.1, C50.1, C51.1, C52.1, C53.1, C54.1, C55.1, C56.1, D31.C, Q13.2, Q14.4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
- net 3.3V4: now also C46.1, C47.1, C48.1, C49.1, C50.1, D29.C, Q25.2, Q26.4; no longer C62.1, C63.1, C64.1, C65.1, C66.1, C67.1, C68.1, C69.1, C70.1, D39.C, Q17.2, Q18.4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
- net 3.3V5: now also C56.1, C57.1, C58.1, C59.1, C60.1, D35.C, Q31.2, Q32.4; no longer C76.1, C77.1, C78.1, C79.1, C80.1, C81.1, C82.1, C83.1, C84.1, D47.C, Q21.2, Q22.4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
- net 3.3V_VREG1: now also C12.1, C13.1, Q6.3, Q8.1, U1.1; no longer C16.1, C17.1, Q2.3, Q4.1, U6.1
- net 3.3V_VREG2: now also C22.1, C23.1, Q13.3, Q14.1, U3.1; no longer C30.1, C31.1, Q10.1, Q9.3, U11.1
- net 3.3V_VREG3: now also C32.1, C33.1, Q19.3, Q20.1, U4.1; no longer C44.1, C45.1, Q13.3, Q14.1, U16.1
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Routing:
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- added copper zone on layer 1, net N$102
- added copper zone on layer 1, net N$25
- added copper zone on layer 1, net N$37
- added copper zone on layer 1, net N$45
- added copper zone on layer 1, net N$56
- added copper zone on layer 1, net N$64
- added copper zone on layer 1, net N$75
- added copper zone on layer 1, net N$83
- added copper zone on layer 1, net N$94
- removed copper zone on layer 1, net N$105 (its old number)
- removed copper zone on layer 1, net N$126
- removed copper zone on layer 1, net N$29 (its old number)
- removed copper zone on layer 1, net N$42
- removed copper zone on layer 1, net N$50
- removed copper zone on layer 1, net N$63
- removed copper zone on layer 1, net N$71
- removed copper zone on layer 1, net N$84
- removed copper zone on layer 1, net N$92
- removed copper zone on layer 1, net SHLD10
- removed copper zone on layer 16, net SHLD10
- removed copper zone on layer 1, net SHLD11
- removed copper zone on layer 16, net SHLD11
- removed copper zone on layer 1, net SHLD6
- removed copper zone on layer 16, net SHLD6
- removed copper zone on layer 1, net SHLD7
- removed copper zone on layer 16, net SHLD7
- removed copper zone on layer 1, net SHLD8
- removed copper zone on layer 16, net SHLD8
- removed copper zone on layer 1, net SHLD9
- removed copper zone on layer 16, net SHLD9
- removed copper zone on layer 1, net VCC
- removed copper zone on layer 1, net VCC1
- removed copper zone on layer 1, net VCC2
- removed copper zone on layer 1, net VCC3
- removed copper zone on layer 1, net VCC4
- removed copper zone on layer 1, net VCC5
- removed copper zone on layer 1, net V_USB_1
- removed copper zone on layer 1, net V_USB_2
- removed copper zone on layer 1, net V_USB_3
- removed copper zone on layer 1, net V_USB_4
- removed copper zone on layer 1, net V_USB_5
- removed copper zone on layer 1, net V_USB_6
Other:
- board text added: "v12"
- board text removed: "v11"
